File: PCB/PID_TEMPERATURE_KICAD.kicad_pcb (KiCad board)
At the start: 2 copper layers, 160 x 102 mm, 74 parts, among them J1 EXT_Supply, J11 BUTTON_2, J12 BUTTON_1, J13 Keyboard1, J14 Keyboard2, J2 LCD 1602 2.54mm, J3 Screw_Terminal_01x05, J4 FAN, J5 Screw_Terminal_01x05, J6 Screw_Terminal_01x05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

Commit message: Project: fixing LED names order
Parts:
- D1: value RED -> GREEN
- D4: value GREEN -> RED
Connections:
- D2 pad 2: /STM_RUNNING -> /REG_MODE
- D4 pad 2: /REG_MODE -> /STM_RUNNING
- R2 pad 1: Net-(D1-K) -> Net-(D4-K)
- R3 pad 1: Net-(D2-K) -> Net-(D3-K)
- R4 pad 1: Net-(D3-K) -> Net-(D2-K)
- R5 pad 1: Net-(D4-K) -> Net-(D1-K)
- U1 pad 32: /STM_RUNNING -> /REG_MODE
- U1 pad 38: /REG_MODE -> /STM_RUNNING
Routing:
- net /STM_RUNNING: track 81.2 -> 101.7 mm
- net /REG_MODE: track 101.7 -> 81.2 mm
Changed lines of the file:
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@@
 			)
 		)
-		(property "Value" "GREEN"
+		(property "Value" "RED"
 			(at 1.27 2.96 270)
 			(layer "F.Fab")
@@
 			(layers "*.Cu" "*.Mask")
 			(remove_unused_layers no)
-			(net 22 "/REG_MODE")
+			(net 18 "/STM_RUNNING")
 			(pinfunction "A")
 			(pintype "passive")
@@
 			(layers "F.Cu" "F.Mask" "F.Paste")
 			(roundrect_rratio 0.2083333333)
-			(net 23 "Net-(D4-K)")
+			(net 17 "Net-(D1-K)")
 			(pintype "passive")
 		)
@@
 			(layers "*.Cu" "*.Mask")
 			(remove_unused_layers no)
-			(net 18 "/STM_RUNNING")
+			(net 22 "/REG_MODE")
 			(pinfunction "A")
 			(pintype "passive")
@@
 			(layers "F.Cu" "F.Mask" "F.Paste")
 			(roundrect_rratio 0.25)
-			(net 18 "/STM_RUNNING")
+			(net 22 "/REG_MODE")
 			(pinfunction "PA11")
 			(pintype "bidirectional")
@@
 			(layers "F.Cu" "F.Mask" "F.Paste")
 			(roundrect_rratio 0.25)
-			(net 22 "/REG_MODE")
+			(net 18 "/STM_RUNNING")
 			(pinfunction "PA15")
 			(pintype "bidirectional")
@@
 			(layers "F.Cu" "F.Mask" "F.Paste")
 			(roundrect_rratio 0.2083333333)
-			(net 19 "Net-(D2-K)")
+			(net 21 "Net-(D3-K)")
 			(pintype "passive")
 		)
@@
 			(layers "F.Cu" "F.Mask" "F.Paste")
 			(roundrect_rratio 0.2083333333)
-			(net 21 "Net-(D3-K)")
+			(net 19 "Net-(D2-K)")
 			(pintype "passive")
 		)
@@
 			(layers "F.Cu" "F.Mask" "F.Paste")
 			(roundrect_rratio 0.2083333333)
-			(net 17 "Net-(D1-K)")
+			(net 23 "Net-(D4-K)")
 			(pintype "passive")
 		)
@@
 			)
 		)
-		(property "Value" "RED"
+		(property "Value" "GREEN"
 			(at 1.27 2.96 270)
 			(layer "F.Fab")
@@
 	)
 	(segment
-		(start 139 90.25)
-		(end 142.41 90.25)
+		(start 137.0875 86.8375)
+		(end 137.0875 84.8325)
 		(width 0.3)
 		(layer "F.Cu")
@@
 	)
 	(segment
-		(start 142.41 90.25)
-		(end 144.01 88.65)
+		(start 137.0875 84.8325)
+		(end 137.46 84.46)
 		(width 0.3)
 		(layer "F.Cu")
@@
 	)
 	(segment
-		(start 144.01 88.65)
-		(end 144.03 88.65)
-		(width 0.2)
+		(start 137.46 84.46)
+		(end 137.51 84.46)
+		(width 0.3)
 		(layer "F.Cu")
 		(net 18)
 	)
 	(segment
-		(start 144.03 88.65)
-		(end 144.03 88.63)
-		(width 0.2)
+		(start 137.51 84.46)
+		(end 137.51 84.41)
+		(width 0.3)
 		(layer "F.Cu")
 		(net 18)
 	)
 	(segment
-		(start 144.03 88.63)
-		(end 144.08 88.58)
-		(width 0.2)
+		(start 137.51 84.41)
+		(end 137.52 84.4)
+		(width 0.3)
 		(layer "F.Cu")
 		(net 18)
 	)
 	(via
-		(at 144.03 88.65)
+		(at 137.51 84.46)
 		(size 0.6)
 		(drill 0.3)
@@
 	)
 	(segment
-		(start 163.525 58.735)
-		(end 193.275 58.735)
+		(start 162.29 55.22)
+		(end 205.47 55.22)
 		(width 0.3)
 		(layer "B.Cu")
@@
 	)
 	(segment
-		(start 162.21 83.52)
-		(end 162.21 60.05)
+		(start 205.47 55.22)
+		(end 207.275 57.025)
 		(width 0.3)
 		(layer "B.Cu")
@@
 	)
 	(segment
-		(start 162.21 60.05)
-		(end 163.525 58.735)
+		(start 160.24 57.27)
+		(end 162.29 55.22)
 		(width 0.3)
 		(layer "B.Cu")
@@
 	)
 	(segment
-		(start 157.08 88.65)
-		(end 162.21 83.52)
+		(start 158.15 84.46)
+		(end 160.24 82.37)
 		(width 0.3)
 		(layer "B.Cu")
@@
 	)
 	(segment
-		(start 144.03 88.65)
-		(end 157.08 88.65)
+		(start 137.51 84.46)
+		(end 158.15 84.46)
+		(width 0.3)
+		(layer "B.Cu")
+		(net 18)
+	)
+	(segment
+		(start 207.275 57.025)
+		(end 207.275 58.735)
+		(width 0.3)
+		(layer "B.Cu")
+		(net 18)
+	)
+	(segment
+		(start 160.24 82.37)
+		(end 160.24 57.27)
 		(width 0.3)
 		(layer "B.Cu")
@@
 	)
 	(segment
-		(start 137.0875 86.8375)
-		(end 137.0875 84.8325)
+		(start 139 90.25)
+		(end 142.41 90.25)
 		(width 0.3)
 		(layer "F.Cu")
@@
 	)
 	(segment
-		(start 137.0875 84.8325)
-		(end 137.46 84.46)
+		(start 142.41 90.25)
+		(end 144.01 88.65)
 		(width 0.3)
 		(layer "F.Cu")
@@
 	)
 	(segment
-		(start 137.46 84.46)
-		(end 137.51 84.46)
-		(width 0.3)
+		(start 144.01 88.65)
+		(end 144.03 88.65)
+		(width 0.2)
 		(layer "F.Cu")
 		(net 22)
 	)
 	(segment
-		(start 137.51 84.46)
-		(end 137.51 84.41)
-		(width 0.3)
+		(start 144.03 88.65)
+		(end 144.03 88.63)
+		(width 0.2)
 		(layer "F.Cu")
 		(net 22)
 	)
 	(segment
-		(start 137.51 84.41)
-		(end 137.52 84.4)
-		(width 0.3)
+		(start 144.03 88.63)
+		(end 144.08 88.58)
+		(width 0.2)
 		(layer "F.Cu")
 		(net 22)
 	)
 	(via
-		(at 137.51 84.46)
+		(at 144.03 88.65)
 		(size 0.6)
 		(drill 0.3)
@@
 	)
 	(segment
-		(start 162.29 55.22)
-		(end 205.47 55.22)
-		(width 0.3)
-		(layer "B.Cu")
-		(net 22)
-	)
-	(segment
-		(start 205.47 55.22)
-		(end 207.275 57.025)
-		(width 0.3)
-		(layer "B.Cu")
-		(net 22)
-	)
-	(segment
-		(start 160.24 57.27)
-		(end 162.29 55.22)
+		(start 163.525 58.735)
+		(end 193.275 58.735)
 		(width 0.3)
 		(layer "B.Cu")
@@
 	)
 	(segment
-		(start 158.15 84.46)
-		(end 160.24 82.37)
+		(start 162.21 83.52)
+		(end 162.21 60.05)
 		(width 0.3)
 		(layer "B.Cu")
@@
 	)
 	(segment
-		(start 137.51 84.46)
-		(end 158.15 84.46)
+		(start 162.21 60.05)
+		(end 163.525 58.735)
 		(width 0.3)
 		(layer "B.Cu")
@@
 	)
 	(segment
-		(start 207.275 57.025)
-		(end 207.275 58.735)
+		(start 157.08 88.65)
+		(end 162.21 83.52)
 		(width 0.3)
 		(layer "B.Cu")
@@
 	)
 	(segment
-		(start 160.24 82.37)
-		(end 160.24 57.27)
+		(start 144.03 88.65)
+		(end 157.08 88.65)
 		(width 0.3)
 		(layer "B.Cu")
