File: PCB/PID_TEMPERATURE_KICAD.kicad_sch (KiCad schematic)
At the start: 60 parts, among them J1 EXT_Supply, J11 BUTTON_2, J12 BUTTON_1, J13 Keyboard1, J14 Keyboard2, J2 LCD 1602 2.54mm, J3 Screw_Terminal_01x05, J4 FAN, J5 Screw_Terminal_01x05, J6 Screw_Terminal_01x05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

Commit message: project: fixing LED color description
Parts:
- D1: value RED -> GREEN
- D4: value GREEN -> RED
Connections:
- net at R5.1: now also D1.1 (K); no longer D4.1 (K)
- net at D2.1 (K): now also R4.1; no longer R3.1
- net at D3.1 (K): now also R3.1; no longer R4.1
- net at R2.1: now also D4.1 (K); no longer D1.1 (K)
Other:
- moved on the sheet: D1, D2, D3, D4
Changed lines of the file:
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@@
 	(wire
 		(pts
+			(xy 187.96 39.37) (xy 187.96 41.91)
+		)
+		(stroke
+			(width 0)
+			(type default)
+		)
+	)
+	(wire
+		(pts
 			(xy 99.06 31.75) (xy 102.87 31.75)
 		)
@@
 	(wire
 		(pts
-			(xy 201.93 41.91) (xy 201.93 39.37)
-		)
-		(stroke
-			(width 0)
-			(type default)
-		)
-	)
-	(wire
-		(pts
 			(xy 209.55 124.46) (xy 207.01 124.46)
 		)
@@
 	(wire
 		(pts
-			(xy 40.64 86.36) (xy 57.15 86.36)
+			(xy 201.93 39.37) (xy 201.93 41.91)
 		)
 		(stroke
@@
 	(wire
 		(pts
-			(xy 151.13 48.26) (xy 148.59 48.26)
+			(xy 40.64 86.36) (xy 57.15 86.36)
 		)
 		(stroke
@@
 	(wire
 		(pts
-			(xy 67.31 154.94) (xy 67.31 158.75)
+			(xy 151.13 48.26) (xy 148.59 48.26)
 		)
 		(stroke
@@
 	(wire
 		(pts
-			(xy 113.03 83.82) (xy 115.57 83.82)
+			(xy 67.31 154.94) (xy 67.31 158.75)
 		)
 		(stroke
@@
 	(wire
 		(pts
-			(xy 109.22 161.29) (xy 116.84 161.29)
+			(xy 113.03 83.82) (xy 115.57 83.82)
 		)
 		(stroke
@@
 	(wire
 		(pts
-			(xy 215.9 49.53) (xy 215.9 54.61)
+			(xy 109.22 161.29) (xy 116.84 161.29)
 		)
 		(stroke
@@
 	(wire
 		(pts
-			(xy 187.96 41.91) (xy 187.96 39.37)
+			(xy 215.9 49.53) (xy 215.9 54.61)
 		)
 		(stroke
@@
 	(wire
 		(pts
+			(xy 215.9 39.37) (xy 215.9 41.91)
+		)
+		(stroke
+			(width 0)
+			(type default)
+		)
+	)
+	(wire
+		(pts
 			(xy 58.42 173.99) (xy 58.42 177.8)
 		)
@@
 	(wire
 		(pts
-			(xy 173.99 39.37) (xy 173.99 41.91)
+			(xy 62.23 39.37) (xy 63.5 39.37)
 		)
 		(stroke
@@
 	(wire
 		(pts
-			(xy 62.23 39.37) (xy 63.5 39.37)
+			(xy 101.6 154.94) (xy 101.6 161.29)
 		)
 		(stroke
@@
 	(wire
 		(pts
-			(xy 101.6 154.94) (xy 101.6 161.29)
+			(xy 173.99 39.37) (xy 173.99 41.91)
 		)
 		(stroke
@@
 	(wire
 		(pts
-			(xy 215.9 41.91) (xy 215.9 39.37)
-		)
-		(stroke
-			(width 0)
-			(type default)
-		)
-	)
-	(wire
-		(pts
 			(xy 157.48 160.02) (xy 148.59 160.02)
 		)
@@
 	)
 	(label "CONFIG_MODE"
-		(at 201.93 31.75 90)
+		(at 187.96 31.75 90)
 		(effects
 			(font
@@
 	)
 	(label "STM_RUNNING"
-		(at 187.96 31.75 90)
+		(at 201.93 31.75 90)
 		(effects
 			(font
@@
 	)
 	(label "REG_MODE"
-		(at 215.9 31.75 90)
+		(at 173.99 31.75 90)
 		(effects
 			(font
@@
 	(symbol
 		(lib_id "Device:LED")
-		(at 187.96 35.56 90)
+		(at 201.93 35.56 90)
 		(unit 1)
 		(exclude_from_sim no)
@@
 		(fields_autoplaced yes)
 		(property "Reference" "D2"
-			(at 191.77 35.8774 90)
+			(at 205.74 35.8774 90)
 			(effects
 				(font
@@
 		)
 		(property "Value" "YELLOW"
-			(at 191.77 38.4174 90)
+			(at 205.74 38.4174 90)
 			(effects
 				(font
@@
 		)
 		(property "Footprint" "LED_THT:LED_D3.0mm"
-			(at 187.96 35.56 0)
+			(at 201.93 35.56 0)
 			(effects
 				(font
@@
 		)
 		(property "Datasheet" "~"
-			(at 187.96 35.56 0)
+			(at 201.93 35.56 0)
 			(effects
 				(font
@@
 		)
 		(property "Description" "Light emitting diode"
-			(at 187.96 35.56 0)
+			(at 201.93 35.56 0)
 			(effects
 				(font
@@
 	(symbol
 		(lib_id "Device:LED")
-		(at 201.93 35.56 90)
+		(at 187.96 35.56 90)
 		(unit 1)
 		(exclude_from_sim no)
@@
 		(fields_autoplaced yes)
 		(property "Reference" "D3"
-			(at 205.74 35.8774 90)
+			(at 191.77 35.8774 90)
 			(effects
 				(font
@@
 		)
 		(property "Value" "YELLOW"
-			(at 205.74 38.4174 90)
+			(at 191.77 38.4174 90)
 			(effects
 				(font
@@
 		)
 		(property "Footprint" "LED_THT:LED_D3.0mm"
-			(at 201.93 35.56 0)
+			(at 187.96 35.56 0)
 			(effects
 				(font
@@
 		)
 		(property "Datasheet" "~"
-			(at 201.93 35.56 0)
+			(at 187.96 35.56 0)
 			(effects
 				(font
@@
 		)
 		(property "Description" "Light emitting diode"
-			(at 201.93 35.56 0)
+			(at 187.96 35.56 0)
 			(effects
 				(font
@@
 	(symbol
 		(lib_id "Device:LED")
-		(at 173.99 35.56 90)
+		(at 215.9 35.56 90)
 		(unit 1)
 		(exclude_from_sim no)
@@
 		(fields_autoplaced yes)
 		(property "Reference" "D1"
-			(at 177.8 35.8774 90)
+			(at 219.71 35.8774 90)
 			(effects
 				(font
@@
 			)
 		)
-		(property "Value" "RED"
-			(at 177.8 38.4174 90)
+		(property "Value" "GREEN"
+			(at 219.71 38.4174 90)
 			(effects
 				(font
@@
 		)
 		(property "Footprint" "LED_THT:LED_D3.0mm"
-			(at 173.99 35.56 0)
+			(at 215.9 35.56 0)
 			(effects
 				(font
@@
 		)
 		(property "Datasheet" "~"
-			(at 173.99 35.56 0)
+			(at 215.9 35.56 0)
 			(effects
 				(font
@@
 		)
 		(property "Description" "Light emitting diode"
-			(at 173.99 35.56 0)
+			(at 215.9 35.56 0)
 			(effects
 				(font
@@
 	(symbol
 		(lib_id "power:+3.3V")
-		(at 173.99 31.75 0)
+		(at 215.9 31.75 0)
 		(unit 1)
 		(exclude_from_sim no)
@@
 		(dnp no)
 		(property "Reference" "#PWR053"
-			(at 173.99 35.56 0)
+			(at 215.9 35.56 0)
 			(effects
 				(font
@@
 		)
 		(property "Value" "+3.3V"
-			(at 173.9899 27.94 90)
+			(at 215.8999 27.94 90)
 			(effects
 				(font
@@
 		)
 		(property "Footprint" ""
-			(at 173.99 31.75 0)
+			(at 215.9 31.75 0)
 			(effects
 				(font
@@
 		)
 		(property "Datasheet" ""
-			(at 173.99 31.75 0)
+			(at 215.9 31.75 0)
 			(effects
 				(font
@@
 		)
 		(property "Description" "Power symbol creates a global label with name \"+3.3V\""
-			(at 173.99 31.75 0)
+			(at 215.9 31.75 0)
 			(effects
 				(font
@@
 	(symbol
 		(lib_id "Device:LED")
-		(at 215.9 35.56 90)
+		(at 173.99 35.56 90)
 		(unit 1)
 		(exclude_from_sim no)
@@
 		(fields_autoplaced yes)
 		(property "Reference" "D4"
-			(at 219.71 35.8774 90)
+			(at 177.8 35.8774 90)
 			(effects
 				(font
@@
 			)
 		)
-		(property "Value" "GREEN"
-			(at 219.71 38.4174 90)
+		(property "Value" "RED"
+			(at 177.8 38.4174 90)
 			(effects
 				(font
@@
 		)
 		(property "Footprint" "LED_THT:LED_D3.0mm"
-			(at 215.9 35.56 0)
+			(at 173.99 35.56 0)
 			(effects
 				(font
@@
 		)
 		(property "Datasheet" "~"
-			(at 215.9 35.56 0)
+			(at 173.99 35.56 0)
 			(effects
 				(font
@@
 		)
 		(property "Description" "Light emitting diode"
-			(at 215.9 35.56 0)
+			(at 173.99 35.56 0)
 			(effects
 				(font

Commit message: Project: fixing LED names order
Connections:
- net REG_MODE: now also D2.2 (A), U1.32 (PA11); no longer D4.2 (A), U1.38 (PA15)
- net STM_RUNNING: now also D4.2 (A), U1.38 (PA15); no longer D2.2 (A), U1.32 (PA11)
Changed lines of the file:
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@@
 		)
 	)
-	(label "REG_MODE"
+	(label "STM_RUNNING"
 		(at 151.13 76.2 0)
 		(effects
@@
 		)
 	)
-	(label "STM_RUNNING"
+	(label "REG_MODE"
 		(at 201.93 31.75 90)
 		(effects
@@
 		)
 	)
-	(label "STM_RUNNING"
+	(label "REG_MODE"
 		(at 151.13 66.04 0)
 		(effects
@@
 		)
 	)
-	(label "REG_MODE"
+	(label "STM_RUNNING"
 		(at 173.99 31.75 90)
 		(effects
